File: bot_ander.kicad_sch (KiCad schematic)
At the start: 3 parts

Commit message: Finish initial schematic
Parts:
- removed U? (x2): ULN2003, symbol Transistor_Array:ULN2003
- added A?: Pololu_Breakout_A4988, Module:Pololu_Breakout-16_15.2x20.3mm, symbol Driver_Motor:Pololu_Breakout_A4988
- added C?: 10uF_e, Capacitor_THT:CP_Radial_D5.0mm_P2.50mm, symbol Device:C_Polarized_US
- added D?: LED, symbol Device:LED
- added M?: Motor_DC, symbol Motor:Motor_DC
- added M?: Motor_Servo, symbol Motor:Motor_Servo
- added M?: Stepper_Motor_bipolar, symbol Motor:Stepper_Motor_bipolar
- added Q? (x3): 2N7000, Package_TO_SOT_THT:TO-92_Inline, symbol Transistor_FET:2N7000
- added R? (x2): R, symbol Device:R
- added U?: LTR-303ALS-01, OptoDevice:Lite-On_LTR-303ALS-01, symbol Sensor_Optical:LTR-303ALS-01
Connections:
- net LED_CNTL: now reaches A?.10 (D7)
- net LED_CNTL: now also Q?.2 (G)
- net SDA: now reaches A?.23 (A4)
- net SDA: now also U?.6 (SDA)
- net SCL: now reaches A?.24 (A5)
- net SCL: now also U?.4 (SCL)
- net +5V: now reaches A?.27 (+5V)
- net +5V: now also A?.2 (VDD), D?.2 (A), U?.1 (VDD)
- net +12V: now reaches A?.30 (VIN)
- net +12V: now also A?.8 (VMOT), C?.1, M?.2 (+), Q?.3 (D)
- net STEP: now reaches A?.5 (D2)
- net STEP: now also A?.15 (STEP)
- net DIR: now reaches A?.6 (D3)
- net DIR: now also A?.16 (DIR)
- net MOT_CNTL: now reaches A?.7 (D4)
- net MOT_CNTL: now also Q?.2 (G)
- net SERVO_PWM: now reaches A?.8 (D5)
- net SERVO_PWM: now also M?.1 (PWM)
- net MOT_CNTL_NOT: now reaches A?.9 (D6)
- net MOT_CNTL_NOT: now also Q?.2 (G)
- new net: Q?.1 (S), R?.1
- new net: Q?.3 (D), R?.2
- new net: D?.1 (K), R?.1
- new net: A?.13 (~{RESET}), A?.14 (~{SLEEP})
- new net: A?.3 (1B), M?.2 (-)
- new net: A?.4 (1A), M?.1
- new net: A?.5 (2A), M?.3
- new net: A?.6 (2B), M?.4
- new net: M?.1 (+), Q?.1 (S), Q?.3 (D)
- new net GND: A?.1 (GND), A?.7 (GND), C?.2, M?.2 (-), M?.3 (-), Q?.1 (S), R?.2, U?.3 (GND)
- no-connect marks 0 -> 7
Other:
- note added: "Arduino Nano"
- note added: "DC Motor Half-Bridge"
- note added: "Servo Motor"
- note added: "Stepper Motor/Driver"
- note added: "UV LED"
- note added: "UV Sensor"
- moved on the sheet: A?
